File: IO.kicad_sch (KiCad schematic)
At the start: 38 parts, among them J10 5VIN, J11 Conn_02x08_Counter_Clockwise, J2 Conn_01x06, J3 Conn_01x06, J4 Conn_01x06, J5 Conn_01x06, J6 Conn_01x06, J7 Conn_01x06, J8 Conn_01x06, J9 Conn_01x06

Commit message: Initial design
Parts:
- added J12: Conn_02x08_Counter_Clockwise, Connector_PinHeader_2.54mm:PinHeader_2x08_P2.54mm_Vertical, symbol Connector_Generic:Conn_02x08_Counter_Clockwise
- added TP15, TP16, TP17, TP18, TP19, TP20: TestPoint, TestPoint:TestPoint_Pad_D2.0mm, symbol Connector:TestPoint
- C50, C51, C52, C60, C61, C62, C63, C64: Digikey PN (none) -> 1276-1044-1-ND; Unit Cost (none) -> 0.044
- C65: footprint Capacitor_THT:C_Radial_D6.3mm_H7.0mm_P2.50mm -> Capacitor_THT:C_Radial_D5.0mm_H7.0mm_P2.00mm; Digikey PN (none) -> P814-ND; Unit Cost (none) -> 0.27
- D7: footprint (none) -> Diode_SMD:D_SOD-923; Digikey PN (none) -> ESD9X5.0ST5GOSCT-ND; Unit Cost (none) -> 0.17
- D8: footprint (none) -> Diode_SMD:D_SOD-123; Digikey PN (none) -> SS24FLCT-ND; Unit Cost (none) -> 0.42
- F1: footprint (none) -> Fuse:Fuse_0603_1608Metric; Digikey PN (none) -> 5923-0686F7000-01CT-ND; Unit Cost (none) -> 0.45
- J10: footprint (none) -> Connector_JST:JST_XH_B2B-XH-A_1x02_P2.50mm_Vertical; Digikey PN (none) -> 455-B2B-XH-A-ND; Unit Cost (none) -> 0.10
- J11: footprint (none) -> Connector_PinHeader_2.54mm:PinHeader_2x08_P2.54mm_Vertical; Digikey PN (none) -> 4627-PH254V-216-6TBKG126-ND; Unit Cost (none) -> 0.34
- J2, J3, J4, J5, J6, J7, J8, J9: footprint (none) -> Connector_JST:JST_GH_SM06B-GHS-TB_1x06-1MP_P1.25mm_Horizontal; Digikey PN (none) -> 455-BM06B-GHS-TBTCT-ND; Unit Cost (none) -> 0.47
- R38, R41, R42, R45, R46, R49, R68, R71: now not fitted; now left out of the parts list
- R39, R40, R43, R44, R47, R48, R69, R70: Digikey PN (none) -> 311-10KLDCT-ND; Unit Cost (none) -> 0.028
Connections:
- net +3.3V: now also J12.10 (Pin_10), J12.7 (Pin_7)
- net GND: now also J12.8 (Pin_8), J12.9 (Pin_9)
- net I2S.DATA0: now also TP17.1
- net I2S.DATA1: now also TP18.1
- net I2S.DATA2: now also TP19.1
- net I2S.DATA3: now also TP20.1
- net I2S.SCK: now also TP15.1
- net I2S.WS: now also TP16.1
- new net FT.CS: J12.13 (Pin_13)
- new net FT.HOLD: J12.11 (Pin_11)
- new net FT.MISO: J12.14 (Pin_14)
- new net FT.MOSI: J12.15 (Pin_15)
- new net FT.RESETN: J12.12 (Pin_12)
- new net FT.SCLK: J12.16 (Pin_16)
- new net JTAG.TCK: J12.3 (Pin_3)
- new net JTAG.TDI: J12.4 (Pin_4)
- new net JTAG.TDO: J12.5 (Pin_5)
- new net JTAG.TMS: J12.6 (Pin_6)
- new net UART.RX: J12.2 (Pin_2)
- new net UART.TX: J12.1 (Pin_1)
Other:
- note added: "Programming"

Commit message: Added ethernet
Parts:
- added J14: Conn_01x10, Connector_PinHeader_2.54mm:PinHeader_1x10_P2.54mm_Vertical, symbol Connector_Generic:Conn_01x10
- TP15, TP16, TP17, TP18, TP19, TP20: now left out of the parts list
Connections:
- net +3.3V: now also J14.1 (Pin_1)
- net GND: now also J14.2 (Pin_2)
- new net GPIO0: J14.3 (Pin_3)
- new net GPIO1: J14.4 (Pin_4)
- new net GPIO2: J14.5 (Pin_5)
- new net GPIO3: J14.6 (Pin_6)
- new net GPIO4: J14.7 (Pin_7)
- new net GPIO5: J14.8 (Pin_8)
- new net GPIO6: J14.9 (Pin_9)
- new net GPIO7: J14.10 (Pin_10)
Other:
- note added: "GPIO"

Commit message: Cleanup
Other:
- title: (none) -> I/O
Changed lines of the file:
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@@
 	(generator_version "10.0")
 	(paper "A4")
+	(title_block
+		(title "I/O")
+		(date "2026-09-19")
+	)
 	(rectangle
 		(start 132.08 55.88)

Commit message: Annotated schematic
Parts:
- renumbered C60 to C47, C50 to C48, C61 to C49, C63 to C50, C52 to C51, C51 to C52, C62 to C53, C64 to C54, C65 to C55, D8 to D7, D7 to D8, J11 to J10, J12 to J11, J10 to J12, J14 to J13, J4 to J3, J6 to J4, J8 to J5, J3 to J6, J5 to J7, J7 to J8, R38 to R49, R39 to R50, R42 to R51, R43 to R52, R46 to R53, R47 to R54, R68 to R55, R69 to R56, R40 to R57, R41 to R58, R44 to R59, R45 to R60, R48 to R61, R49 to R62, R70 to R63, R71 to R64, TP15 to TP28, TP18 to TP29, TP16 to TP30, TP19 to TP31, TP17 to TP32, TP20 to TP33

Commit message: Started module-level layout
Parts:
- removed J10, J11: Conn_02x08_Counter_Clockwise, Connector_PinHeader_2.54mm:PinHeader_2x08_P2.54mm_Vertical, symbol Connector_Generic:Conn_02x08_Counter_Clockwise
- added J10, J11: Conn_02x08_Odd_Even, Connector_PinHeader_2.54mm:PinHeader_2x08_P2.54mm_Vertical, symbol Connector_Generic:Conn_02x08_Odd_Even
- J2, J3, J4, J5, J6, J7, J8, J9: footprint Connector_JST:JST_GH_SM06B-GHS-TB_1x06-1MP_P1.25mm_Horizontal -> Connector_JST:JST_GH_BM06B-GHS-TBT_1x06-1MP_P1.25mm_Vertical
- TP29: renamed from TP28; footprint TestPoint:TestPoint_Pad_D2.0mm -> TestPoint:TestPoint_Pad_D1.0mm
- TP30: renamed from TP29; footprint TestPoint:TestPoint_Pad_D2.0mm -> TestPoint:TestPoint_Pad_D1.0mm
- TP31: renamed from TP30; footprint TestPoint:TestPoint_Pad_D2.0mm -> TestPoint:TestPoint_Pad_D1.0mm
- TP32: renamed from TP31; footprint TestPoint:TestPoint_Pad_D2.0mm -> TestPoint:TestPoint_Pad_D1.0mm
- TP33: renamed from TP32; footprint TestPoint:TestPoint_Pad_D2.0mm -> TestPoint:TestPoint_Pad_D1.0mm
- TP34: renamed from TP33; footprint TestPoint:TestPoint_Pad_D2.0mm -> TestPoint:TestPoint_Pad_D1.0mm
- renumbered C47 to C48, C48 to C49, C49 to C50, C50 to C51, C51 to C52, C52 to C53, C53 to C54, C54 to C55, C55 to C56, F1 to F2, R49 to R51, R50 to R52, R51 to R53, R52 to R54, R53 to R55, R54 to R56, R55 to R57, R56 to R58, R57 to R59, R58 to R60, R59 to R61, R60 to R62, R61 to R63, R62 to R64, R63 to R65, R64 to R66
Connections:
- net +3.3V: now also J11.13 (Pin_13), J11.14 (Pin_14)
- net ADC0: now also J10.15 (Pin_15)
- net ADC1: now also J10.13 (Pin_13)
- net ADC2: now also J10.11 (Pin_11)
- net ADC3: now also J10.9 (Pin_9)
- net ADC4: now also J10.7 (Pin_7)
- net ADC5: now also J10.5 (Pin_5)
- net ADC6: now also J10.3 (Pin_3)
- net ADC7: now also J10.1 (Pin_1)
- net FT.CS: now also J11.8 (Pin_8)
- net FT.HOLD: now also J11.12 (Pin_12)
- net FT.MISO: now also J11.6 (Pin_6)
- net FT.MOSI: now also J11.4 (Pin_4)
- net FT.RESETN: now also J11.10 (Pin_10)
- net FT.SCLK: now also J11.2 (Pin_2)
- net GND: now also J10.10 (Pin_10), J10.12 (Pin_12), J10.14 (Pin_14), J10.16 (Pin_16), J10.2 (Pin_2), J10.4 (Pin_4), J10.6 (Pin_6), J10.8 (Pin_8), J11.15 (Pin_15), J11.16 (Pin_16)
- net JTAG.TCK: now also J11.5 (Pin_5)
- net JTAG.TDI: now also J11.7 (Pin_7)
- net JTAG.TDO: now also J11.9 (Pin_9)
- net JTAG.TMS: now also J11.11 (Pin_11)
- net UART.RX: now also J11.3 (Pin_3)
- net UART.TX: now also J11.1 (Pin_1)

Commit message: More layout
Parts:
- D7: footprint Diode_SMD:D_SOD-123 -> Diode_SMD:D_SMA; Digikey PN SS24FLCT-ND -> 5399-SS32CT-ND; Unit Cost 0.42 -> 0.10
- D8: footprint Diode_SMD:D_SOD-923 -> Diode_SMD:D_SMA; Digikey PN ESD9X5.0ST5GOSCT-ND -> 5399-SMAJ6.0ACT-ND
Changed lines of the file:
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@@
 			)
 		)
-		(property "Footprint" "Diode_SMD:D_SOD-123"
+		(property "Footprint" "Diode_SMD:D_SMA"
 			(at 153.67 41.91 0)
 			(hide yes)
@@
 			)
 		)
-		(property "Digikey PN" "SS24FLCT-ND"
+		(property "Digikey PN" "5399-SS32CT-ND"
 			(at 153.67 41.91 90)
 			(hide yes)
@@
 			)
 		)
-		(property "Unit Cost" "0.42"
+		(property "Unit Cost" "0.10"
 			(at 153.67 41.91 90)
 			(hide yes)
@@
 			)
 		)
-		(property "Footprint" "Diode_SMD:D_SOD-923"
+		(property "Footprint" "Diode_SMD:D_SMA"
 			(at 161.29 41.91 0)
 			(hide yes)
@@
 			)
 		)
-		(property "Digikey PN" "ESD9X5.0ST5GOSCT-ND"
+		(property "Digikey PN" "5399-SMAJ6.0ACT-ND"
 			(at 161.29 41.91 90)
 			(hide yes)

Commit message: More layout
Connections:
- net GND: now also J12.1 (Pin_1); no longer J12.2 (Pin_2)
- net at D7.1 (K), D8.1 (A1), F2.1: now also J12.2 (Pin_2); no longer J12.1 (Pin_1)
Changed lines of the file:
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@@
 	(wire
 		(pts
+			(xy 171.45 40.64) (xy 173.99 40.64)
+		)
+		(stroke
+			(width 0)
+			(type default)
+		)
+	)
+	(wire
+		(pts
 			(xy 91.44 41.91) (xy 91.44 43.18)
 		)
@@
 	(wire
 		(pts
+			(xy 171.45 43.18) (xy 173.99 43.18)
+		)
+		(stroke
+			(width 0)
+			(type default)
+		)
+	)
+	(wire
+		(pts
 			(xy 156.21 74.93) (xy 162.56 74.93)
 		)
@@
 	(wire
 		(pts
-			(xy 173.99 43.18) (xy 171.45 43.18)
-		)
-		(stroke
-			(width 0)
-			(type default)
-		)
-	)
-	(wire
-		(pts
 			(xy 127 50.8) (xy 127 52.07)
 		)
@@
 	(wire
 		(pts
-			(xy 173.99 40.64) (xy 171.45 40.64)
-		)
-		(stroke
-			(width 0)
-			(type default)
-		)
-	)
-	(wire
-		(pts
 			(xy 78.74 85.09) (xy 78.74 86.36)
 		)
@@
 	(symbol
 		(lib_id "Connector_Generic:Conn_01x02")
-		(at 179.07 40.64 0)
+		(at 179.07 43.18 0)
+		(mirror x)
 		(unit 1)
 		(body_style 1)
@@
 		(in_pos_files yes)
 		(dnp no)
-		(fields_autoplaced yes)
 		(property "Reference" "J12"
-			(at 181.61 40.6399 0)
+			(at 181.61 43.1801 0)
 			(show_name no)
 			(do_not_autoplace no)
@@
 		)
 		(property "Value" "5VIN"
-			(at 181.61 43.1799 0)
+			(at 181.61 40.6401 0)
 			(show_name no)
 			(do_not_autoplace no)
@@
 		)
 		(property "Footprint" "Connector_JST:JST_XH_B2B-XH-A_1x02_P2.50mm_Vertical"
-			(at 179.07 40.64 0)
+			(at 179.07 43.18 0)
 			(hide yes)
 			(show_name no)
@@
 		)
 		(property "Datasheet" ""
-			(at 179.07 40.64 0)
+			(at 179.07 43.18 0)
 			(hide yes)
 			(show_name no)
@@
 		)
 		(property "Description" "Generic connector, single row, 01x02, script generated (kicad-library-utils/schlib/autogen/connector/)"
-			(at 179.07 40.64 0)
+			(at 179.07 43.18 0)
 			(hide yes)
 			(show_name no)
@@
 		)
 		(property "Digikey PN" "455-B2B-XH-A-ND"
-			(at 179.07 40.64 0)
+			(at 179.07 43.18 0)
 			(hide yes)
 			(show_name no)
@@
 		)
 		(property "Unit Cost" "0.10"
-			(at 179.07 40.64 0)
+			(at 179.07 43.18 0)
 			(hide yes)
 			(show_name no)
@@
 		)
 		(property "KLC_S3.3" ""
-			(at 179.07 40.64 0)
+			(at 179.07 43.18 0)
 			(hide yes)
 			(show_name no)
@@
 		)
 		(property "KLC_S4.1" ""
-			(at 179.07 40.64 0)
+			(at 179.07 43.18 0)
 			(hide yes)
 			(show_name no)
