File: IO.kicad_sch (KiCad schematic)
At the start: 46 parts, among them J10 Conn_02x08_Odd_Even, J11 Conn_02x08_Odd_Even, J12 5VIN, J13 Conn_01x10, J2 Conn_01x06, J3 Conn_01x06, J4 Conn_01x06, J5 Conn_01x06, J6 Conn_01x06, J7 Conn_01x06, J8 Conn_01x06, J9 Conn_01x06

Commit message: Added SPI bus buffer
Changed lines of the file:
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@@
 	(rectangle
 		(start 132.08 99.06)
-		(end 240.03 144.78)
+		(end 247.65 144.78)
 		(stroke
 			(width 0)
@@
 		)
 	)
-	(hierarchical_label "FT{SCLK MOSI MISO CS RESETN HOLD}"
+	(hierarchical_label "FT{SCLK MOSI MISO CS RESETN HOLD CDONE}"
 		(shape bidirectional)
 		(at 200.66 133.35 0)

Commit message: Finalized
Parts:
- C48, C49, C50, C51, C52, C53, C54, C55: Digikey PN 1276-1044-1-ND -> 1276-1045-1-ND; Unit Cost 0.044 -> 0.041
Changed lines of the file:
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@@
 			)
 		)
-		(property "Digikey PN" "1276-1044-1-ND"
+		(property "Digikey PN" "1276-1045-1-ND"
 			(at 43.18 115.57 0)
 			(hide yes)
@@
 			)
 		)
-		(property "Unit Cost" "0.044"
+		(property "Unit Cost" "0.041"
 			(at 43.18 115.57 0)
 			(hide yes)
@@
 			)
 		)
-		(property "Digikey PN" "1276-1044-1-ND"
+		(property "Digikey PN" "1276-1045-1-ND"
 			(at 36.83 46.99 0)
 			(hide yes)
@@
 			)
 		)
-		(property "Unit Cost" "0.044"
+		(property "Unit Cost" "0.041"
 			(at 36.83 46.99 0)
 			(hide yes)
@@
 			)
 		)
-		(property "Digikey PN" "1276-1044-1-ND"
+		(property "Digikey PN" "1276-1045-1-ND"
 			(at 91.44 149.86 0)
 			(hide yes)
@@
 			)
 		)
-		(property "Unit Cost" "0.044"
+		(property "Unit Cost" "0.041"
 			(at 91.44 149.86 0)
 			(hide yes)
@@
 			)
 		)
-		(property "Digikey PN" "1276-1044-1-ND"
+		(property "Digikey PN" "1276-1045-1-ND"
 			(at 91.44 46.99 0)
 			(hide yes)
@@
 			)
 		)
-		(property "Unit Cost" "0.044"
+		(property "Unit Cost" "0.041"
 			(at 91.44 46.99 0)
 			(hide yes)
@@
 			)
 		)
-		(property "Digikey PN" "1276-1044-1-ND"
+		(property "Digikey PN" "1276-1045-1-ND"
 			(at 91.44 115.57 0)
 			(hide yes)
@@
 			)
 		)
-		(property "Unit Cost" "0.044"
+		(property "Unit Cost" "0.041"
 			(at 91.44 115.57 0)
 			(hide yes)
@@
 			)
 		)
-		(property "Digikey PN" "1276-1044-1-ND"
+		(property "Digikey PN" "1276-1045-1-ND"
 			(at 43.18 81.28 0)
 			(hide yes)
@@
 			)
 		)
-		(property "Unit Cost" "0.044"
+		(property "Unit Cost" "0.041"
 			(at 43.18 81.28 0)
 			(hide yes)
@@
 			)
 		)
-		(property "Digikey PN" "1276-1044-1-ND"
+		(property "Digikey PN" "1276-1045-1-ND"
 			(at 43.18 149.86 0)
 			(hide yes)
@@
 			)
 		)
-		(property "Unit Cost" "0.044"
+		(property "Unit Cost" "0.041"
 			(at 43.18 149.86 0)
 			(hide yes)
@@
 			)
 		)
-		(property "Digikey PN" "1276-1044-1-ND"
+		(property "Digikey PN" "1276-1045-1-ND"
 			(at 91.44 82.55 0)
 			(hide yes)
@@
 			)
 		)
-		(property "Unit Cost" "0.044"
+		(property "Unit Cost" "0.041"
 			(at 91.44 82.55 0)
 			(hide yes)
