File: Ethernet.kicad_sch (KiCad schematic)
At the start: 23 parts, among them J13 RJ45_Halo_HFJ11-x2450E-LxxRL, U9 LAN8720A

Commit message: Cleanup
Parts:
- added TP34, TP35, TP36, TP37, TP38, TP39, TP40, TP41, TP42, TP43, TP44: TestPoint, TestPoint:TestPoint_Pad_D2.0mm, symbol Connector:TestPoint
Connections:
- net RMII.CRS_DV: now also TP40.1
- net RMII.INT: now also TP44.1
- net RMII.MDC: now also TP42.1
- net RMII.MDIO: now also TP41.1
- net RMII.RSTN: now also TP43.1
- net RMII.RXD0: now also TP37.1
- net RMII.RXD1: now also TP38.1
- net RMII.RXER: now also TP39.1
- net RMII.TXD0: now also TP34.1
- net RMII.TXD1: now also TP35.1
- net RMII.TXEN: now also TP36.1
Other:
- note added: "Config Pullups"
- note added: "PHY"
- note added: "RJ45"
- note added: "RMII Testpoints"
- title: (none) -> Ethernet
- moved on the sheet: C66, C67, C70, C71, J13, R74, R75, R76, R77, R82, R83, R84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

Commit message: Annotated schematic
Parts:
- renumbered C71 to C66, C70 to C67, C67 to C68, C66 to C69, C69 to C70, C68 to C71, J13 to J14, R76 to R73, R77 to R74, R86 to R75, R75 to R76, R85 to R77, R74 to R78, R84 to R79, R83 to R80, R82 to R81, R78 to R82, R73 to R83, R79 to R84, R80 to R85, R81 to R86

Commit message: Started module-level layout
Parts:
- TP35: renamed from TP34; footprint TestPoint:TestPoint_Pad_D2.0mm -> TestPoint:TestPoint_Pad_D1.0mm
- TP36: renamed from TP35; footprint TestPoint:TestPoint_Pad_D2.0mm -> TestPoint:TestPoint_Pad_D1.0mm
- TP37: renamed from TP36; footprint TestPoint:TestPoint_Pad_D2.0mm -> TestPoint:TestPoint_Pad_D1.0mm
- TP38: renamed from TP37; footprint TestPoint:TestPoint_Pad_D2.0mm -> TestPoint:TestPoint_Pad_D1.0mm
- TP39: renamed from TP38; footprint TestPoint:TestPoint_Pad_D2.0mm -> TestPoint:TestPoint_Pad_D1.0mm
- TP40: renamed from TP39; footprint TestPoint:TestPoint_Pad_D2.0mm -> TestPoint:TestPoint_Pad_D1.0mm
- TP41: renamed from TP40; footprint TestPoint:TestPoint_Pad_D2.0mm -> TestPoint:TestPoint_Pad_D1.0mm
- TP42: renamed from TP41; footprint TestPoint:TestPoint_Pad_D2.0mm -> TestPoint:TestPoint_Pad_D1.0mm
- TP43: renamed from TP42; footprint TestPoint:TestPoint_Pad_D2.0mm -> TestPoint:TestPoint_Pad_D1.0mm
- TP44: renamed from TP43; footprint TestPoint:TestPoint_Pad_D2.0mm -> TestPoint:TestPoint_Pad_D1.0mm
- TP45: renamed from TP44; footprint TestPoint:TestPoint_Pad_D2.0mm -> TestPoint:TestPoint_Pad_D1.0mm
- renumbered C66 to C67, C67 to C68, C68 to C69, C69 to C70, C70 to C71, C71 to C72, R73 to R75, R74 to R76, R75 to R77, R76 to R78, R77 to R79, R78 to R80, R79 to R81, R80 to R82, R81 to R83, R82 to R84, R83 to R85, R84 to R86, R85 to R87, R86 to R88, U9 to U10

Commit message: Routing done
Parts:
- removed TP35, TP36, TP37, TP38, TP39, TP40, TP41, TP42, TP43, TP44, TP45: TestPoint, TestPoint:TestPoint_Pad_D1.0mm, symbol Connector:TestPoint
Other:
- note removed: "RMII Testpoints"
