File: fpga_pcb.kicad_sch (KiCad schematic)
At the start: 4 parts

Commit message: Added SPI bus buffer
Other:
- sheet FPGA ports: added FT{SCLK MOSI MISO CS RESETN HOLD CDONE}; removed FT{SCLK MOSI MISO CS RESETN HOLD}
- sheet IO ports: added FT{SCLK MOSI MISO CS RESETN HOLD CDONE}; removed FT{SCLK MOSI MISO CS RESETN HOLD}
- sheet USB ports: added FT{SCLK MOSI MISO CS RESETN HOLD CDONE}; removed FT{SCLK MOSI MISO CS RESETN HOLD}
Changed lines of the file:
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@@
 	)
 	(sheet
-		(at 21.59 86.36)
-		(size 39.37 25.4)
+		(at 13.97 86.36)
+		(size 46.99 25.4)
 		(exclude_from_sim no)
 		(in_bom yes)
@@
 		)
 		(property "Sheetname" "USB"
-			(at 21.59 85.6484 0)
+			(at 13.97 85.6484 0)
 			(show_name no)
 			(do_not_autoplace no)
@@
 		)
 		(property "Sheetfile" "USB.kicad_sch"
-			(at 21.59 112.3446 0)
+			(at 13.97 112.3446 0)
 			(show_name no)
 			(do_not_autoplace no)
@@
 			)
 		)
-		(pin "FT{SCLK MOSI MISO CS RESETN HOLD}" bidirectional
+		(pin "FT{SCLK MOSI MISO CS RESETN HOLD CDONE}" bidirectional
 			(at 60.96 101.6 0)
 			(effects
@@
 			)
 		)
-		(pin "FT{SCLK MOSI MISO CS RESETN HOLD}" bidirectional
+		(pin "FT{SCLK MOSI MISO CS RESETN HOLD CDONE}" bidirectional
 			(at 77.47 101.6 180)
 			(effects
@@
 	(sheet
 		(at 237.49 88.9)
-		(size 43.18 38.1)
+		(size 46.99 38.1)
 		(exclude_from_sim no)
 		(in_bom yes)
@@
 			)
 		)
-		(pin "FT{SCLK MOSI MISO CS RESETN HOLD}" bidirectional
+		(pin "FT{SCLK MOSI MISO CS RESETN HOLD CDONE}" bidirectional
 			(at 237.49 115.57 180)
 			(effects
