File: FPGA.kicad_sch (KiCad schematic)
At the start: 69 parts, among them SW1 SW_Push, SW2 SW_Push, U2 23AA02M-IST, Y1 ECS-2520MV-500-xx

Commit message: Added SPI bus buffer
Connections:
- net CDONE renamed FT.CDONE
Changed lines of the file:
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@@
 	)
 	(bus_entry
+		(at 60.96 170.18)
+		(size 2.54 2.54)
+		(stroke
+			(width 0)
+			(type default)
+		)
+	)
+	(bus_entry
 		(at 71.12 181.61)
 		(size -2.54 2.54)
@@
 	(bus
 		(pts
-			(xy 67.31 170.18) (xy 68.58 170.18)
+			(xy 59.69 170.18) (xy 68.58 170.18)
 		)
 		(stroke
@@
 	(wire
 		(pts
+			(xy 63.5 172.72) (xy 73.66 172.72)
+		)
+		(stroke
+			(width 0)
+			(type default)
+		)
+	)
+	(wire
+		(pts
 			(xy 45.72 43.18) (xy 45.72 44.45)
 		)
@@
 		)
 	)
-	(label "CDONE"
+	(label "FT.CDONE"
 		(at 124.46 180.34 0)
 		(effects
@@
 		)
 	)
-	(label "CDONE"
+	(label "FT.CDONE"
 		(at 114.3 93.98 180)
 		(effects
@@
 		)
 	)
+	(label "FT.CDONE"
+		(at 73.66 172.72 180)
+		(effects
+			(font
+				(size 1.27 1.27)
+			)
+			(justify right bottom)
+		)
+	)
 	(label "JTAG.TCK"
 		(at 34.29 147.32 90)
@@
 		)
 	)
-	(hierarchical_label "FT{SCLK MOSI MISO CS RESETN HOLD}"
+	(hierarchical_label "FT{SCLK MOSI MISO CS RESETN HOLD CDONE}"
 		(shape bidirectional)
-		(at 67.31 170.18 180)
+		(at 59.69 170.18 180)
 		(effects
 			(font

Commit message: Finalized
Parts:
- C11, C14, C4, C8: Digikey PN 1276-1044-1-ND -> 1276-1045-1-ND; Unit Cost 0.044 -> 0.041
Changed lines of the file:
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@@
 			)
 		)
-		(property "Digikey PN" "1276-1044-1-ND"
+		(property "Digikey PN" "1276-1045-1-ND"
 			(at 63.5 72.39 0)
 			(hide yes)
@@
 			)
 		)
-		(property "Unit Cost" "0.044"
+		(property "Unit Cost" "0.041"
 			(at 63.5 72.39 0)
 			(hide yes)
@@
 			)
 		)
-		(property "Digikey PN" "1276-1044-1-ND"
+		(property "Digikey PN" "1276-1045-1-ND"
 			(at 76.2 72.39 0)
 			(hide yes)
@@
 			)
 		)
-		(property "Unit Cost" "0.044"
+		(property "Unit Cost" "0.041"
 			(at 76.2 72.39 0)
 			(hide yes)
@@
 			)
 		)
-		(property "Digikey PN" "1276-1044-1-ND"
+		(property "Digikey PN" "1276-1045-1-ND"
 			(at 88.9 72.39 0)
 			(hide yes)
@@
 			)
 		)
-		(property "Unit Cost" "0.044"
+		(property "Unit Cost" "0.041"
 			(at 88.9 72.39 0)
 			(hide yes)
@@
 			)
 		)
-		(property "Digikey PN" "1276-1044-1-ND"
+		(property "Digikey PN" "1276-1045-1-ND"
 			(at 50.8 72.39 0)
 			(hide yes)
@@
 			)
 		)
-		(property "Unit Cost" "0.044"
+		(property "Unit Cost" "0.041"
 			(at 50.8 72.39 0)
 			(hide yes)
