File: Power.kicad_sch (KiCad schematic)
At the start: 27 parts, among them U3 TPS62A02APDDC, U4 TLV75733PDBV, U5 TPS2116DRL

Commit message: Finalized
Parts:
- C25, C73: Digikey PN 1276-1044-1-ND -> 1276-1045-1-ND; Unit Cost 0.044 -> 0.041
Changed lines of the file:
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@@
 			)
 		)
-		(property "Digikey PN" "1276-1044-1-ND"
+		(property "Digikey PN" "1276-1045-1-ND"
 			(at 82.55 123.19 0)
 			(hide yes)
@@
 			)
 		)
-		(property "Unit Cost" "0.044"
+		(property "Unit Cost" "0.041"
 			(at 82.55 123.19 0)
 			(hide yes)
@@
 			)
 		)
-		(property "Digikey PN" "1276-1044-1-ND"
+		(property "Digikey PN" "1276-1045-1-ND"
 			(at 45.72 74.93 0)
 			(hide yes)
@@
 			)
 		)
-		(property "Unit Cost" "0.044"
+		(property "Unit Cost" "0.041"
 			(at 45.72 74.93 0)
 			(hide yes)
